File: Platine/HM-LC-Bl1-FM-DC.kicad_pcb (KiCad board)
At the start: 2 copper layers, 53.1 x 26.9 mm, 32 parts, among them J2 FTDI, J4 Reset, K1 OMRONG6S-2, K2 OMRONG6S-2, Q1 BC817, Q2 BC817, SW2 Config, U1 ATMEGA328P-AU, U2 CC1101, U3 AM1S-2403S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

Commit message: update to 2.1
fix mirrored footprint of X2
Parts:
- C7: value 100n -> 3.3u 35V
- R21, R23: value R -> 10k
- R22, R24: value R -> 47
- moved X2 7.51 mm to (76.7, 90.8), turned to 0 degrees
- moved R21 4.15 mm to (77.6, 98.6), turned to 0 degrees
- moved R23 4.08 mm to (77.9, 91.4), turned to 0 degrees
- moved R22 2.17 mm to (77.6, 96.8)
Connections:
- K2 pad 10: (no net) -> Net-(K2-Pad10)
- K2 pad 3: (no net) -> Net-(K2-Pad3)
- K2 pad 4: (no net) -> Net-(K2-Pad4)
- K2 pad 5: (no net) -> Net-(K2-Pad5)
- U1 pad 11: (no net) -> Net-(U1-Pad11)
- U1 pad 13: (no net) -> Net-(U1-Pad13)
- U1 pad 19: (no net) -> Net-(U1-Pad19)
- U1 pad 22: (no net) -> Net-(U1-Pad22)
- U1 pad 25: (no net) -> Net-(U1-Pad25)
- U1 pad 26: (no net) -> Net-(U1-Pad26)
- U1 pad 27: (no net) -> Net-(U1-Pad27)
- U1 pad 28: (no net) -> Net-(U1-Pad28)
- U1 pad 7: (no net) -> Net-(U1-Pad7)
- U1 pad 8: (no net) -> Net-(U1-Pad8)
- U1 pad 9: (no net) -> Net-(U1-Pad9)
- U2 pad 6: (no net) -> Net-(U2-Pad6)
- X2 pad L1: /UP -> /DOWN
- X2 pad L3: /DOWN -> /UP
Routing:
- net VCC: track 19.6 -> 16.8 mm
- net /D6: track 58.1 -> 59.0 mm
- net /UP: track 5.91 -> 5.29 mm
Other:
- board text added: "CC BY-NC-SA 4.0"
- board text added: "HM-LC-Bl1-FM-DC stan23 V2.1 10/18"
- board text removed: "HM-LC-Bl1-FM-DC stan23 V2.0 07/18"
